File: ATO.sch (KiCad schematic (older format))
At the start: 19 parts, among them J1 Pump Out, J2 Switch, J3 Power, Q1 Q_NMOS_GDSD, Q2 Q_PJFET_SGD, Q3 Q_NJFET_DGS, Q4 Q_PJFET_SGD, SW1 Reset, SW2 Fill

Commit message: Added cap on power input and other tweaks.
Parts:
- added C2: CP, Capacitor_THT:C_Disc_D9.0mm_W2.5mm_P5.00mm, symbol Device:CP
- Q1: value Q_NMOS_GDSD -> NFET
- Q2, Q4: value Q_PJFET_SGD -> PFET
- Q3: value Q_NJFET_DGS -> NFET
Connections:
- wire segments 36 -> 38
Changed lines of the file:
@@
 P 6750 2600
 F 0 "Q4" H 6940 2646 50  0000 L CNN
-F 1 "Q_PJFET_SGD" H 6940 2555 50  0000 L CNN
+F 1 "PFET" H 6940 2555 50  0000 L CNN
 F 2 "Package_TO_SOT_THT:TO-92_HandSolder" H 6950 2700 50  0001 C CNN
 F 3 "~" H 6750 2600 50  0001 C CNN
@@
 Connection ~ 6850 2300
 Wire Wire Line
-	6850 2300 8150 2300
+	6850 2300 7500 2300
 Wire Wire Line
 	6550 2600 6450 2600
@@
 P 5500 3350
 F 0 "Q3" H 5691 3396 50  0000 L CNN
-F 1 "Q_NJFET_DGS" H 5691 3305 50  0000 L CNN
+F 1 "NFET" H 5691 3305 50  0000 L CNN
 F 2 "Package_TO_SOT_THT:TO-92_HandSolder" H 5700 3450 50  0001 C CNN
 F 3 "~" H 5500 3350 50  0001 C CNN
@@
 P 5100 2750
 F 0 "Q2" H 5291 2796 50  0000 L CNN
-F 1 "Q_PJFET_SGD" H 5291 2705 50  0000 L CNN
+F 1 "PFET" H 5291 2705 50  0000 L CNN
 F 2 "Package_TO_SOT_THT:TO-92_HandSolder" H 5300 2850 50  0001 C CNN
 F 3 "~" H 5100 2750 50  0001 C CNN
@@
 P 4600 3350
 F 0 "Q1" H 4888 3396 50  0000 L CNN
-F 1 "Q_NMOS_GDSD" H 4888 3305 50  0000 L CNN
+F 1 "NFET" H 4888 3305 50  0000 L CNN
 F 2 "Package_TO_SOT_THT:TO-251-3-1EP_Horizontal_TabDown" H 4800 3450 50  0001 C CNN
 F 3 "~" H 4600 3350 50  0001 C CNN
@@
 	6400 2300 6850 2300
 $Comp
-L Graphic:Logo_Open_Hardware_Small #LOGO?
+L Graphic:Logo_Open_Hardware_Small #LOGO1
 U 1 1 610A9FB5
 P 3350 1800
-F 0 "#LOGO?" H 3350 2075 50  0001 C CNN
+F 0 "#LOGO1" H 3350 2075 50  0001 C CNN
 F 1 "Logo_Open_Hardware_Small" H 3350 1575 50  0001 C CNN
 F 2 "Symbol:OSHW-Symbol_8.9x8mm_SilkScreen" H 3350 1800 50  0001 C CNN
@@
 	1    0    0    -1
 $EndComp
+$Comp
+L Device:CP C2
+U 1 1 6105BE75
+P 7500 2450
+F 0 "C2" H 7618 2496 50  0000 L CNN
+F 1 "CP" H 7618 2405 50  0000 L CNN
+F 2 "Capacitor_THT:C_Disc_D9.0mm_W2.5mm_P5.00mm" H 7538 2300 50  0001 C CNN
+F 3 "~" H 7500 2450 50  0001 C CNN
+	1    7500 2450
+	1    0    0    -1
+$EndComp
+Connection ~ 7500 2300
+Wire Wire Line
+	7500 2300 8150 2300
+$Comp
+L power:GND #PWR0102
+U 1 1 6105C8FF
+P 7500 2700
+F 0 "#PWR0102" H 7500 2450 50  0001 C CNN
+F 1 "GND" H 7505 2527 50  0000 C CNN
+F 2 "" H 7500 2700 50  0001 C CNN
+F 3 "" H 7500 2700 50  0001 C CNN
+	1    7500 2700
+	1    0    0    -1
+$EndComp
+Wire Wire Line
+	7500 2700 7500 2600
 $EndSCHEMATC
